File: currentSink.sch (KiCad schematic (older format))
At the start: 0 parts

Commit message: adding preliminary schematic
Parts:
- added C? (x2): C, symbol C
- added P? (x2): CONN_01X01, symbol CONN_01X01
- added Q?: MOSFET_N, symbol MOSFET_N
- added R? (x2): R, symbol R
- added U?: LMV358, symbol LMV358
- added U?: MCP4922-E/SL, SO14, symbol MCP4922-E/SL
- added U?: TC1016, symbol TC1016
Connections:
- net labels added: GND
- wire segments 0 -> 21
Changed lines of the file:
@@
 LIBS:contrib
 LIBS:valves
+LIBS:currentSink
+LIBS:currentSink-cache
 EELAYER 25 0
 EELAYER END
@@
 Comment4 ""
 $EndDescr
+$Comp
+L LMV358 U?
+U 1 1 5520C82C
+P 5850 3100
+F 0 "U?" H 5800 3300 60  0000 L CNN
+F 1 "LMV358" H 5800 2850 60  0000 L CNN
+F 2 "" H 5850 3100 60  0000 C CNN
+F 3 "" H 5850 3100 60  0000 C CNN
+	1    5850 3100
+	1    0    0    -1
+$EndComp
+$Comp
+L GND #PWR?
+U 1 1 5520C877
+P 7700 4700
+F 0 "#PWR?" H 7700 4450 60  0001 C CNN
+F 1 "GND" H 7700 4550 60  0000 C CNN
+F 2 "" H 7700 4700 60  0000 C CNN
+F 3 "" H 7700 4700 60  0000 C CNN
+	1    7700 4700
+	1    0    0    -1
+$EndComp
+$Comp
+L R R?
+U 1 1 5520C893
+P 7700 4300
+F 0 "R?" V 7780 4300 50  0000 C CNN
+F 1 "R" V 7707 4301 50  0000 C CNN
+F 2 "" V 7630 4300 30  0000 C CNN
+F 3 "" H 7700 4300 30  0000 C CNN
+	1    7700 4300
+	1    0    0    -1
+$EndComp
+$Comp
+L MOSFET_N Q?
+U 1 1 5520C8BE
+P 7600 3100
+F 0 "Q?" H 7610 3270 50  0000 R CNN
+F 1 "MOSFET_N" H 7550 2950 50  0000 R CNN
+F 2 "" H 7600 3100 60  0000 C CNN
+F 3 "" H 7600 3100 60  0000 C CNN
+	1    7600 3100
+	1    0    0    -1
+$EndComp
+$Comp
+L R R?
+U 1 1 5520C94C
+P 6850 3100
+F 0 "R?" V 6930 3100 50  0000 C CNN
+F 1 "R" V 6857 3101 50  0000 C CNN
+F 2 "" V 6780 3100 30  0000 C CNN
+F 3 "" H 6850 3100 30  0000 C CNN
+	1    6850 3100
+	0    1    1    0
+$EndComp
+$Comp
+L GND #PWR?
+U 1 1 5520CA34
+P 5750 3600
+F 0 "#PWR?" H 5750 3350 60  0001 C CNN
+F 1 "GND" H 5750 3450 60  0000 C CNN
+F 2 "" H 5750 3600 60  0000 C CNN
+F 3 "" H 5750 3600 60  0000 C CNN
+	1    5750 3600
+	1    0    0    -1
+$EndComp
+$Comp
+L CONN_01X01 P?
+U 1 1 5520CA7E
+P 9550 4650
+F 0 "P?" H 9550 4750 50  0000 C CNN
+F 1 "CONN_01X01" V 9650 4650 50  0000 C CNN
+F 2 "" H 9550 4650 60  0000 C CNN
+F 3 "" H 9550 4650 60  0000 C CNN
+	1    9550 4650
+	1    0    0    -1
+$EndComp
+$Comp
+L CONN_01X01 P?
+U 1 1 5520CAE0
+P 9650 1950
+F 0 "P?" H 9650 2050 50  0000 C CNN
+F 1 "CONN_01X01" V 9750 1950 50  0000 C CNN
+F 2 "" H 9650 1950 60  0000 C CNN
+F 3 "" H 9650 1950 60  0000 C CNN
+	1    9650 1950
+	1    0    0    -1
+$EndComp
+$Comp
+L MCP4922-E/SL U?
+U 1 1 5520CE1D
+P 2650 2850
+F 0 "U?" H 2800 3250 40  0000 L BNN
+F 1 "MCP4922-E/SL" H 2800 3200 40  0000 L BNN
+F 2 "SO14" H 2650 2850 30  0000 C CIN
+F 3 "" H 2650 2850 60  0000 C CNN
+	1    2650 2850
+	1    0    0    -1
+$EndComp
+Wire Wire Line
+	5350 3000 3200 3000
+Wire Wire Line
+	5350 2950 5350 3000
+Connection ~ 7700 4650
+Wire Wire Line
+	9350 4650 7700 4650
+Wire Wire Line
+	5750 3500 5750 3600
+Connection ~ 7700 3850
+Wire Wire Line
+	5350 3850 7700 3850
+Wire Wire Line
+	5350 3200 5350 3850
+Wire Wire Line
+	6350 3100 6600 3100
+Wire Wire Line
+	7100 3100 7400 3100
+Wire Wire Line
+	7700 3300 7700 4050
+Wire Wire Line
+	7700 4550 7700 4700
+$Comp
+L TC1016 U?
+U 1 1 5520CF99
+P 6800 2000
+F 0 "U?" H 6950 1804 60  0000 C CNN
+F 1 "TC1016" H 6800 2200 60  0000 C CNN
+F 2 "" H 6800 2000 60  0000 C CNN
+F 3 "" H 6800 2000 60  0000 C CNN
+	1    6800 2000
+	-1   0    0    -1
+$EndComp
+Wire Wire Line
+	2550 1950 6400 1950
+Wire Wire Line
+	5750 1950 5750 2700
+Wire Wire Line
+	2550 2400 2550 1950
+Connection ~ 5750 1950
+$Comp
+L GND #PWR?
+U 1 1 5520D273
+P 6800 2550
+F 0 "#PWR?" H 6800 2300 60  0001 C CNN
+F 1 "GND" H 6800 2400 60  0000 C CNN
+F 2 "" H 6800 2550 60  0000 C CNN
+F 3 "" H 6800 2550 60  0000 C CNN
+	1    6800 2550
+	1    0    0    -1
+$EndComp
+Wire Wire Line
+	6800 2550 6800 2250
+Wire Wire Line
+	7200 1950 9450 1950
+Wire Wire Line
+	7700 2900 7700 1950
+Connection ~ 7700 1950
+$Comp
+L C C?
+U 1 1 5520D778
+P 7400 2300
+F 0 "C?" H 7450 2400 50  0000 L CNN
+F 1 "C" H 7450 2200 50  0000 L CNN
+F 2 "" H 7438 2150 30  0000 C CNN
+F 3 "" H 7400 2300 60  0000 C CNN
+	1    7400 2300
+	1    0    0    -1
+$EndComp
+$Comp
+L C C?
+U 1 1 5520D7B4
+P 6200 2350
+F 0 "C?" H 6250 2450 50  0000 L CNN
+F 1 "C" H 6250 2250 50  0000 L CNN
+F 2 "" H 6238 2200 30  0000 C CNN
+F 3 "" H 6200 2350 60  0000 C CNN
+	1    6200 2350
+	1    0    0    -1
+$EndComp
+Wire Wire Line
+	6200 2150 6200 1950
+Connection ~ 6200 1950
+Wire Wire Line
+	6200 2550 6800 2550
+Connection ~ 7400 1950
+Wire Wire Line
+	7400 2100 7400 1950
+Wire Wire Line
+	7400 2500 6800 2500
+Connection ~ 6800 2500
+$Comp
+L GND #PWR?
+U 1 1 5520DDF9
+P 2550 3550
+F 0 "#PWR?" H 2550 3300 60  0001 C CNN
+F 1 "GND" H 2550 3400 60  0000 C CNN
+F 2 "" H 2550 3550 60  0000 C CNN
+F 3 "" H 2550 3550 60  0000 C CNN
+	1    2550 3550
+	1    0    0    -1
+$EndComp
+Wire Wire Line
+	2550 3300 2550 3550
 $EndSCHEMATC
