File: currentSink.sch (KiCad schematic (older format))
At the start: 4 parts

Commit message: updated schematic to include a switch for use of an external power source to the circuit
Parts:
- added P?: ExtBatt_Power, symbol CONN_01X02
- added SW?: SWITCH_INV, symbol SWITCH_INV
Connections:
- wire segments 39 -> 51
Other:
- moved on the sheet: P?
Changed lines of the file:
@@
 $EndComp
 $Sheet
-S 5850 2650 1350 1500
+S 5850 2850 1350 1500
 U 55212F37
 F0 "Current Control" 60
 F1 "currentControl.sch" 60
-F2 "DAC_Vb" I L 5850 3000 60
-F3 "Current_Sink-" I R 7200 3700 60
-F4 "Current_Sink+" I R 7200 3000 60
-F5 "FET_Gate" I L 5850 3350 60
+F2 "DAC_Vb" I L 5850 3200 60
+F3 "Current_Sink-" I R 7200 3900 60
+F4 "Current_Sink+" I R 7200 3200 60
+F5 "FET_Gate" I L 5850 3550 60
 $EndSheet
 $Sheet
@@
 $EndComp
 $Sheet
-S 5850 700  1300 1500
+S 5850 950  1300 1500
 U 55216B3A
 F0 "Power Regulation" 60
 F1 "powerRegulation.sch" 60
-F2 "Vin" I R 7150 1400 60
+F2 "Vin" I L 5850 1700 60
 $EndSheet
 $Sheet
@@
 	5850 5400 5500 5400
 Wire Wire Line
-	5500 5400 5500 3350
-Wire Wire Line
-	5500 3350 5850 3350
-Wire Wire Line
-	7200 3700 9450 3700
+	5500 3550 5850 3550
+Wire Wire Line
+	7200 3900 9450 3900
 Wire Wire Line
 	7500 5050 7200 5050
 Wire Wire Line
 	8150 5750 7200 5750
-Connection ~ 8150 3700
 Wire Wire Line
 	4350 4350 4800 4350
 Wire Wire Line
-	4800 4350 4800 3000
-Wire Wire Line
-	4800 3000 5850 3000
+	4800 3200 5850 3200
 Wire Wire Line
 	4350 4750 4800 4750
@@
 	9450 1050 9250 1050
 Wire Wire Line
-	7150 1400 7900 1400
-Wire Wire Line
 	9250 1850 10250 1850
 Wire Wire Line
@@
 Wire Wire Line
 	2300 5500 1500 5500
-Wire Wire Line
-	7500 1400 7500 5050
-Connection ~ 7500 1400
-Wire Wire Line
-	7200 3000 7500 3000
-Connection ~ 7500 3000
-Wire Wire Line
-	8150 3700 8150 5750
 $Comp
 L CONN_01X02 P?
 U 1 1 55229A93
-P 1300 2750
-F 0 "P?" H 1300 2900 50  0000 C CNN
-F 1 "uPower" V 1400 2750 50  0000 C CNN
-F 2 "" H 1300 2750 60  0000 C CNN
-F 3 "" H 1300 2750 60  0000 C CNN
-F 4 "Value" H 1300 2750 60  0001 C CNN "MPN"
-	1    1300 2750
+P 1300 3100
+F 0 "P?" H 1300 3250 50  0000 C CNN
+F 1 "uPower" V 1400 3100 50  0000 C CNN
+F 2 "" H 1300 3100 60  0000 C CNN
+F 3 "" H 1300 3100 60  0000 C CNN
+F 4 "Value" H 1300 3100 60  0001 C CNN "MPN"
+	1    1300 3100
 	-1   0    0    1
 $EndComp
@@
 L GND #PWR?
 U 1 1 55229C45
-P 1900 2350
-F 0 "#PWR?" H 1900 2100 60  0001 C CNN
-F 1 "GND" H 1900 2200 60  0000 C CNN
-F 2 "" H 1900 2350 60  0000 C CNN
-F 3 "" H 1900 2350 60  0000 C CNN
-	1    1900 2350
+P 1900 2700
+F 0 "#PWR?" H 1900 2450 60  0001 C CNN
+F 1 "GND" H 1900 2550 60  0000 C CNN
+F 2 "" H 1900 2700 60  0000 C CNN
+F 3 "" H 1900 2700 60  0000 C CNN
+	1    1900 2700
 	1    0    0    -1
 $EndComp
 Wire Wire Line
-	1500 2700 1500 2150
-Wire Wire Line
-	1500 2150 1900 2150
-Wire Wire Line
-	1900 2150 1900 2350
-Text GLabel 2200 2800 2    60   Input ~ 0
+	1500 3050 1500 2500
+Wire Wire Line
+	1500 2500 1900 2500
+Wire Wire Line
+	1900 2500 1900 2700
+Text GLabel 2200 3150 2    60   Input ~ 0
 3.3V
 Wire Wire Line
-	1500 2800 2200 2800
+	1500 3150 2200 3150
+Wire Wire Line
+	7900 1400 7500 1400
+Wire Wire Line
+	7500 700  7500 5050
+Wire Wire Line
+	7200 3200 7500 3200
+Connection ~ 7500 3200
+Wire Wire Line
+	8150 5750 8150 3900
+Connection ~ 8150 3900
+Wire Wire Line
+	5500 5400 5500 3550
+Wire Wire Line
+	4800 4350 4800 3200
+$Comp
+L SWITCH_INV SW?
+U 1 1 5521E775
+P 4400 1450
+F 0 "SW?" H 4200 1600 50  0000 C CNN
+F 1 "SWITCH_INV" H 4250 1300 50  0000 C CNN
+F 2 "" H 4400 1450 60  0000 C CNN
+F 3 "" H 4400 1450 60  0000 C CNN
+	1    4400 1450
+	0    1    -1   0
+$EndComp
+Wire Wire Line
+	4500 950  4500 700
+Wire Wire Line
+	4500 700  7500 700
+Connection ~ 7500 1400
+Wire Wire Line
+	4400 1950 5150 1950
+Wire Wire Line
+	5150 1950 5150 1700
+Wire Wire Line
+	5150 1700 5850 1700
+$Comp
+L CONN_01X02 P?
+U 1 1 5521ED8A
+P 1300 1400
+F 0 "P?" H 1300 1550 50  0000 C CNN
+F 1 "ExtBatt_Power" V 1400 1400 50  0000 C CNN
+F 2 "" H 1300 1400 60  0000 C CNN
+F 3 "" H 1300 1400 60  0000 C CNN
+	1    1300 1400
+	-1   0    0    1
+$EndComp
+Wire Wire Line
+	1450 1450 3350 1450
+Wire Wire Line
+	3350 1450 3350 700
+Wire Wire Line
+	3350 700  4300 700
+Wire Wire Line
+	4300 700  4300 950
+$Comp
+L GND #PWR?
+U 1 1 5521EED5
+P 1900 950
+F 0 "#PWR?" H 1900 700 60  0001 C CNN
+F 1 "GND" H 1900 800 60  0000 C CNN
+F 2 "" H 1900 950 60  0000 C CNN
+F 3 "" H 1900 950 60  0000 C CNN
+	1    1900 950
+	1    0    0    -1
+$EndComp
+Wire Wire Line
+	1500 1350 1500 750
+Wire Wire Line
+	1500 750  1900 750
+Wire Wire Line
+	1900 750  1900 950
 $EndSCHEMATC

Commit message: updated with association labels
Parts:
- gave numbers to parts that had none: 6
Changed lines of the file:
@@
 $EndDescr
 $Comp
-L CONN_01X01 P?
+L CONN_01X01 P105
 U 1 1 5520CA7E
 P 9650 3700
-F 0 "P?" H 9650 3800 50  0000 C CNN
+F 0 "P105" H 9650 3800 50  0000 C CNN
 F 1 "Load-ve" V 9750 3700 50  0000 C CNN
 F 2 "" H 9650 3700 60  0000 C CNN
@@
 $EndComp
 $Comp
-L CONN_01X01 P?
+L CONN_01X01 P104
 U 1 1 5520CAE0
 P 9650 1050
-F 0 "P?" H 9650 1150 50  0000 C CNN
+F 0 "P104" H 9650 1150 50  0000 C CNN
 F 1 "Load+ve" V 9750 1050 50  0000 C CNN
 F 2 "" H 9650 1050 60  0000 C CNN
@@
 $EndSheet
 $Comp
-L CONN_01X05 P?
+L CONN_01X05 P103
 U 1 1 5521534C
 P 1300 5300
-F 0 "P?" H 1300 5600 50  0000 C CNN
+F 0 "P103" H 1300 5600 50  0000 C CNN
 F 1 "uSignals" V 1400 5300 50  0000 C CNN
 F 2 "" H 1300 5300 60  0000 C CNN
@@
 $EndComp
 $Comp
-L GND #PWR?
+L GND #PWR103
 U 1 1 552165DD
 P 9450 4050
-F 0 "#PWR?" H 9450 3800 60  0001 C CNN
+F 0 "#PWR103" H 9450 3800 60  0001 C CNN
 F 1 "GND" H 9450 3900 60  0000 C CNN
 F 2 "" H 9450 4050 60  0000 C CNN
@@
 	2300 5500 1500 5500
 $Comp
-L CONN_01X02 P?
+L CONN_01X02 P102
 U 1 1 55229A93
 P 1300 3100
-F 0 "P?" H 1300 3250 50  0000 C CNN
+F 0 "P102" H 1300 3250 50  0000 C CNN
 F 1 "uPower" V 1400 3100 50  0000 C CNN
 F 2 "" H 1300 3100 60  0000 C CNN
@@
 $EndComp
 $Comp
-L GND #PWR?
+L GND #PWR102
 U 1 1 55229C45
 P 1900 2700
-F 0 "#PWR?" H 1900 2450 60  0001 C CNN
+F 0 "#PWR102" H 1900 2450 60  0001 C CNN
 F 1 "GND" H 1900 2550 60  0000 C CNN
 F 2 "" H 1900 2700 60  0000 C CNN
@@
 	4800 4350 4800 3200
 $Comp
-L SWITCH_INV SW?
+L SWITCH_INV SW101
 U 1 1 5521E775
 P 4400 1450
-F 0 "SW?" H 4200 1600 50  0000 C CNN
+F 0 "SW101" H 4200 1600 50  0000 C CNN
 F 1 "SWITCH_INV" H 4250 1300 50  0000 C CNN
 F 2 "" H 4400 1450 60  0000 C CNN
@@
 	5150 1700 5850 1700
 $Comp
-L CONN_01X02 P?
+L CONN_01X02 P101
 U 1 1 5521ED8A
 P 1300 1400
-F 0 "P?" H 1300 1550 50  0000 C CNN
+F 0 "P101" H 1300 1550 50  0000 C CNN
 F 1 "ExtBatt_Power" V 1400 1400 50  0000 C CNN
 F 2 "" H 1300 1400 60  0000 C CNN
@@
 	4300 700  4300 950
 $Comp
-L GND #PWR?
+L GND #PWR101
 U 1 1 5521EED5
 P 1900 950
-F 0 "#PWR?" H 1900 700 60  0001 C CNN
+F 0 "#PWR101" H 1900 700 60  0001 C CNN
 F 1 "GND" H 1900 800 60  0000 C CNN
 F 2 "" H 1900 950 60  0000 C CNN
