File: currentRead.sch (KiCad schematic (older format))
At the start: 4 parts

Commit message: updated with association labels
Parts:
- gave numbers to parts that had none: 4
Changed lines of the file:
@@
 $EndDescr
 $Comp
-L ACS711 U?
+L ACS711 U601
 U 1 1 5522578B
 P 5600 3900
-F 0 "U?" H 5900 3504 60  0000 C CNN
+F 0 "U601" H 5900 3504 60  0000 C CNN
 F 1 "ACS711" H 5600 4050 60  0000 C CNN
 F 2 "" H 5600 3900 60  0000 C CNN
@@
 CurrentSink_Out
 $Comp
-L GND #PWR?
+L GND #PWR601
 U 1 1 55225CFE
 P 6100 4500
-F 0 "#PWR?" H 6100 4250 60  0001 C CNN
+F 0 "#PWR601" H 6100 4250 60  0001 C CNN
 F 1 "GND" H 6100 4350 60  0000 C CNN
 F 2 "" H 6100 4500 60  0000 C CNN
@@
 3.3V
 $Comp
-L R R?
+L R R601
 U 1 1 55225D57
 P 6450 4350
-F 0 "R?" V 6530 4350 50  0000 C CNN
+F 0 "R601" V 6530 4350 50  0000 C CNN
 F 1 "10K" V 6457 4351 50  0000 C CNN
 F 2 "" V 6380 4350 30  0000 C CNN
@@
 $EndComp
 $Comp
-L C C?
+L C C601
 U 1 1 55225E4D
 P 6700 3350
-F 0 "C?" H 6750 3450 50  0000 L CNN
+F 0 "C601" H 6750 3450 50  0000 L CNN
 F 1 "100nf" H 6750 3250 50  0000 L CNN
 F 2 "" H 6738 3200 30  0000 C CNN
@@
 $EndComp
 $Comp
-L GND #PWR?
+L GND #PWR602
 U 1 1 55225E9B
 P 6700 3650
-F 0 "#PWR?" H 6700 3400 60  0001 C CNN
+F 0 "#PWR602" H 6700 3400 60  0001 C CNN
 F 1 "GND" H 6700 3500 60  0000 C CNN
 F 2 "" H 6700 3650 60  0000 C CNN
@@
 Connection ~ 6450 3950
 $Comp
-L C C?
+L C C602
 U 1 1 55225FBA
 P 6750 4300
-F 0 "C?" H 6800 4400 50  0000 L CNN
+F 0 "C602" H 6800 4400 50  0000 L CNN
 F 1 "100nf" H 6800 4200 50  0000 L CNN
 F 2 "" H 6788 4150 30  0000 C CNN
@@
 $EndComp
 $Comp
-L GND #PWR?
+L GND #PWR603
 U 1 1 55225FDC
 P 6750 4600
-F 0 "#PWR?" H 6750 4350 60  0001 C CNN
+F 0 "#PWR603" H 6750 4350 60  0001 C CNN
 F 1 "GND" H 6750 4450 60  0000 C CNN
 F 2 "" H 6750 4600 60  0000 C CNN

Commit message: updated schematic with corrected wiring after all passives became disconnected
Changed lines of the file:
@@
 	6350 4050 6350 4750
 Wire Wire Line
-	6350 4750 6450 4750
+	6450 4750 6350 4750
 Wire Wire Line
-	6450 4750 6450 4600
+	6450 4500 6450 4750
 Wire Wire Line
-	6700 3150 6700 3050
+	6700 3050 6700 3200
 Connection ~ 6700 3050
 Wire Wire Line
-	6700 3550 6700 3650
+	6700 3500 6700 3650
 Wire Wire Line
-	6450 4100 6450 3950
+	6450 3950 6450 4200
 Connection ~ 6450 3950
 $Comp
@@
 $EndComp
 Wire Wire Line
-	6750 4500 6750 4600
+	6750 4450 6750 4600
 Wire Wire Line
-	6750 4100 6750 3950
+	6750 3950 6750 4150
 Connection ~ 6750 3950
 $EndSCHEMATC

Commit message: updated current control circuit with voltage divider to increase resolution to 12mA
Changed lines of the file:
@@
 CurrentSink_Out
 $Comp
-L GND #PWR601
+L GND #PWR028
 U 1 1 55225CFE
 P 6100 4500
-F 0 "#PWR601" H 6100 4250 60  0001 C CNN
+F 0 "#PWR028" H 6100 4250 60  0001 C CNN
 F 1 "GND" H 6100 4350 60  0000 C CNN
 F 2 "" H 6100 4500 60  0000 C CNN
@@
 $EndComp
 $Comp
-L GND #PWR602
+L GND #PWR029
 U 1 1 55225E9B
 P 6700 3650
-F 0 "#PWR602" H 6700 3400 60  0001 C CNN
+F 0 "#PWR029" H 6700 3400 60  0001 C CNN
 F 1 "GND" H 6700 3500 60  0000 C CNN
 F 2 "" H 6700 3650 60  0000 C CNN
@@
 	6350 4050 6350 4750
 Wire Wire Line
-	6450 4750 6350 4750
+	6350 4750 6450 4750
 Wire Wire Line
-	6450 4500 6450 4750
+	6450 4750 6450 4500
 Wire Wire Line
 	6700 3050 6700 3200
@@
 $EndComp
 $Comp
-L GND #PWR603
+L GND #PWR030
 U 1 1 55225FDC
 P 6750 4600
-F 0 "#PWR603" H 6750 4350 60  0001 C CNN
+F 0 "#PWR030" H 6750 4350 60  0001 C CNN
 F 1 "GND" H 6750 4450 60  0000 C CNN
 F 2 "" H 6750 4600 60  0000 C CNN

Commit message: updated project with most footprint associations
Parts:
- C601, C602: footprint (none) -> Capacitors_SMD:C_0805_HandSoldering
- R601: footprint (none) -> Resistors_SMD:R_0805_HandSoldering
Changed lines of the file:
@@
 F 0 "U601" H 5900 3504 60  0000 C CNN
 F 1 "ACS711" H 5600 4050 60  0000 C CNN
-F 2 "" H 5600 3900 60  0000 C CNN
+F 2 "" H 5600 3900 60  0001 C CNN
 F 3 "" H 5600 3900 60  0000 C CNN
 	1    5600 3900
@@
 CurrentSink_Out
 $Comp
-L GND #PWR028
+L GND #PWR601
 U 1 1 55225CFE
 P 6100 4500
-F 0 "#PWR028" H 6100 4250 60  0001 C CNN
+F 0 "#PWR601" H 6100 4250 60  0001 C CNN
 F 1 "GND" H 6100 4350 60  0000 C CNN
 F 2 "" H 6100 4500 60  0000 C CNN
@@
 F 0 "R601" V 6530 4350 50  0000 C CNN
 F 1 "10K" V 6457 4351 50  0000 C CNN
-F 2 "" V 6380 4350 30  0000 C CNN
+F 2 "Resistors_SMD:R_0805_HandSoldering" V 6380 4350 30  0001 C CNN
 F 3 "" H 6450 4350 30  0000 C CNN
 	1    6450 4350
@@
 F 0 "C601" H 6750 3450 50  0000 L CNN
 F 1 "100nf" H 6750 3250 50  0000 L CNN
-F 2 "" H 6738 3200 30  0000 C CNN
+F 2 "Capacitors_SMD:C_0805_HandSoldering" H 6738 3200 30  0001 C CNN
 F 3 "" H 6700 3350 60  0000 C CNN
 F 4 "Value" H 6700 3350 60  0001 C CNN "MPN"
@@
 $EndComp
 $Comp
-L GND #PWR029
+L GND #PWR602
 U 1 1 55225E9B
 P 6700 3650
-F 0 "#PWR029" H 6700 3400 60  0001 C CNN
+F 0 "#PWR602" H 6700 3400 60  0001 C CNN
 F 1 "GND" H 6700 3500 60  0000 C CNN
 F 2 "" H 6700 3650 60  0000 C CNN
@@
 F 0 "C602" H 6800 4400 50  0000 L CNN
 F 1 "100nf" H 6800 4200 50  0000 L CNN
-F 2 "" H 6788 4150 30  0000 C CNN
+F 2 "Capacitors_SMD:C_0805_HandSoldering" H 6788 4150 30  0001 C CNN
 F 3 "" H 6750 4300 60  0000 C CNN
 F 4 "Value" H 6750 4300 60  0001 C CNN "MPN"
@@
 $EndComp
 $Comp
-L GND #PWR030
+L GND #PWR603
 U 1 1 55225FDC
 P 6750 4600
-F 0 "#PWR030" H 6750 4350 60  0001 C CNN
+F 0 "#PWR603" H 6750 4350 60  0001 C CNN
 F 1 "GND" H 6750 4450 60  0000 C CNN
 F 2 "" H 6750 4600 60  0000 C CNN

Commit message: association of footprints complete
Parts:
- U601: footprint (none) -> SMD_Packages:SOIC-8-N; MPN (none) -> ACS711KLCTR-12AB-T
Changed lines of the file:
@@
 F 0 "U601" H 5900 3504 60  0000 C CNN
 F 1 "ACS711" H 5600 4050 60  0000 C CNN
-F 2 "" H 5600 3900 60  0001 C CNN
-F 3 "" H 5600 3900 60  0000 C CNN
+F 2 "SMD_Packages:SOIC-8-N" H 5600 3900 60  0001 C CNN
+F 3 "http://www.digikey.com.au/product-search/en?FV=fff4001e%2Cfff801ed%2C401994%2C12040027&k=acs711&mnonly=0&newproducts=0&ColumnSort=0&page=1&stock=1&pbfree=0&rohs=0&quantity=1&ptm=0&fid=0&pageSize=500" H 5600 3900 60  0001 C CNN
+F 4 "ACS711KLCTR-12AB-T" H 5600 3900 60  0001 C CNN "MPN"
 	1    5600 3900
 	1    0    0    -1
@@
 CurrentSink_Out
 $Comp
-L GND #PWR601
+L GND #PWR028
 U 1 1 55225CFE
 P 6100 4500
-F 0 "#PWR601" H 6100 4250 60  0001 C CNN
+F 0 "#PWR028" H 6100 4250 60  0001 C CNN
 F 1 "GND" H 6100 4350 60  0000 C CNN
 F 2 "" H 6100 4500 60  0000 C CNN
@@
 $EndComp
 $Comp
-L GND #PWR602
+L GND #PWR029
 U 1 1 55225E9B
 P 6700 3650
-F 0 "#PWR602" H 6700 3400 60  0001 C CNN
+F 0 "#PWR029" H 6700 3400 60  0001 C CNN
 F 1 "GND" H 6700 3500 60  0000 C CNN
 F 2 "" H 6700 3650 60  0000 C CNN
@@
 $EndComp
 $Comp
-L GND #PWR603
+L GND #PWR030
 U 1 1 55225FDC
 P 6750 4600
-F 0 "#PWR603" H 6750 4350 60  0001 C CNN
+F 0 "#PWR030" H 6750 4350 60  0001 C CNN
 F 1 "GND" H 6750 4450 60  0000 C CNN
 F 2 "" H 6750 4600 60  0000 C CNN

Commit message: updated with some of the frontside tracks
Parts:
- U601: footprint SMD_Packages:SOIC-8-N -> SOIC-8-N
Changed lines of the file:
@@
 F 0 "U601" H 5900 3504 60  0000 C CNN
 F 1 "ACS711" H 5600 4050 60  0000 C CNN
-F 2 "SMD_Packages:SOIC-8-N" H 5600 3900 60  0001 C CNN
+F 2 "SOIC-8-N" H 5600 3900 60  0001 C CNN
 F 3 "http://www.digikey.com.au/product-search/en?FV=fff4001e%2Cfff801ed%2C401994%2C12040027&k=acs711&mnonly=0&newproducts=0&ColumnSort=0&page=1&stock=1&pbfree=0&rohs=0&quantity=1&ptm=0&fid=0&pageSize=500" H 5600 3900 60  0001 C CNN
 F 4 "ACS711KLCTR-12AB-T" H 5600 3900 60  0001 C CNN "MPN"
