File: currentControl.sch (KiCad schematic (older format))
At the start: 9 parts, among them P201 TST, P202 TST, Q201 BUK9575, U201 LMV358

Commit message: association of footprints complete
Parts:
- P201, P202: footprint (none) -> Measurement_Points:Measurement_Point_Round-TH_Small
- Q201: footprint (none) -> Transistors_TO-220:TO-220_FET-GDS_Vertical
- R202: footprint (none) -> Resistors_ThroughHole:Resistor_Horizontal_RM15mm
- U201: footprint (none) -> SMD_Packages:SOIC-8-N
Changed lines of the file:
@@
 $EndDescr
 $Comp
-L GND #PWR206
+L GND #PWR04
 U 1 1 5521A09C
 P 5100 4750
-F 0 "#PWR206" H 5100 4500 60  0001 C CNN
-F 1 "GND" H 5100 4600 60  0000 C CNN
-F 2 "" H 5100 4750 60  0000 C CNN
-F 3 "" H 5100 4750 60  0000 C CNN
-	1    5100 4750
-	1    0    0    -1
-$EndComp
-$Comp
-L GND #PWR202
+F 0 "#PWR04" H 5100 4500 60  0001 C CNN
+F 1 "GND" H 5100 4600 60  0000 C CNN
+F 2 "" H 5100 4750 60  0000 C CNN
+F 3 "" H 5100 4750 60  0000 C CNN
+	1    5100 4750
+	1    0    0    -1
+$EndComp
+$Comp
+L GND #PWR05
 U 1 1 5521A0A9
 P 4300 3850
-F 0 "#PWR202" H 4300 3600 60  0001 C CNN
-F 1 "GND" H 4300 3700 60  0000 C CNN
-F 2 "" H 4300 3850 60  0000 C CNN
-F 3 "" H 4300 3850 60  0000 C CNN
-	1    4300 3850
-	1    0    0    -1
-$EndComp
-$Comp
-L GND #PWR207
+F 0 "#PWR05" H 4300 3600 60  0001 C CNN
+F 1 "GND" H 4300 3700 60  0000 C CNN
+F 2 "" H 4300 3850 60  0000 C CNN
+F 3 "" H 4300 3850 60  0000 C CNN
+	1    4300 3850
+	1    0    0    -1
+$EndComp
+$Comp
+L GND #PWR06
 U 1 1 5521A0D3
 P 5100 4750
-F 0 "#PWR207" H 5100 4500 60  0001 C CNN
-F 1 "GND" H 5100 4600 60  0000 C CNN
-F 2 "" H 5100 4750 60  0000 C CNN
-F 3 "" H 5100 4750 60  0000 C CNN
-	1    5100 4750
-	1    0    0    -1
-$EndComp
-$Comp
-L GND #PWR203
+F 0 "#PWR06" H 5100 4500 60  0001 C CNN
+F 1 "GND" H 5100 4600 60  0000 C CNN
+F 2 "" H 5100 4750 60  0000 C CNN
+F 3 "" H 5100 4750 60  0000 C CNN
+	1    5100 4750
+	1    0    0    -1
+$EndComp
+$Comp
+L GND #PWR07
 U 1 1 5521A0E0
 P 4300 3850
-F 0 "#PWR203" H 4300 3600 60  0001 C CNN
-F 1 "GND" H 4300 3700 60  0000 C CNN
-F 2 "" H 4300 3850 60  0000 C CNN
-F 3 "" H 4300 3850 60  0000 C CNN
-	1    4300 3850
-	1    0    0    -1
-$EndComp
-$Comp
-L GND #PWR208
+F 0 "#PWR07" H 4300 3600 60  0001 C CNN
+F 1 "GND" H 4300 3700 60  0000 C CNN
+F 2 "" H 4300 3850 60  0000 C CNN
+F 3 "" H 4300 3850 60  0000 C CNN
+	1    4300 3850
+	1    0    0    -1
+$EndComp
+$Comp
+L GND #PWR08
 U 1 1 5521A118
 P 5100 4750
-F 0 "#PWR208" H 5100 4500 60  0001 C CNN
-F 1 "GND" H 5100 4600 60  0000 C CNN
-F 2 "" H 5100 4750 60  0000 C CNN
-F 3 "" H 5100 4750 60  0000 C CNN
-	1    5100 4750
-	1    0    0    -1
-$EndComp
-$Comp
-L GND #PWR204
+F 0 "#PWR08" H 5100 4500 60  0001 C CNN
+F 1 "GND" H 5100 4600 60  0000 C CNN
+F 2 "" H 5100 4750 60  0000 C CNN
+F 3 "" H 5100 4750 60  0000 C CNN
+	1    5100 4750
+	1    0    0    -1
+$EndComp
+$Comp
+L GND #PWR09
 U 1 1 5521A125
 P 4300 3850
-F 0 "#PWR204" H 4300 3600 60  0001 C CNN
+F 0 "#PWR09" H 4300 3600 60  0001 C CNN
 F 1 "GND" H 4300 3700 60  0000 C CNN
 F 2 "" H 4300 3850 60  0000 C CNN
@@
 F 0 "U201" H 5150 4450 60  0000 L CNN
 F 1 "LMV358" H 5150 4000 60  0000 L CNN
-F 2 "" H 5200 4250 60  0001 C CNN
+F 2 "SMD_Packages:SOIC-8-N" H 5200 4250 60  0001 C CNN
 F 3 "" H 5200 4250 60  0000 C CNN
 	1    5200 4250
@@
 F 0 "R202" V 7980 5450 50  0000 C CNN
 F 1 ".1" V 7907 5451 50  0000 C CNN
-F 2 "" V 7830 5450 30  0001 C CNN
+F 2 "Resistors_ThroughHole:Resistor_Horizontal_RM15mm" V 7830 5450 30  0001 C CNN
 F 3 "" H 7900 5450 30  0000 C CNN
 F 4 "AC01000001007JA100" V 7900 5450 60  0001 C CNN "MPN"
@@
 F 0 "Q201" H 7810 4420 50  0000 R CNN
 F 1 "BUK9575" H 7750 4100 50  0000 R CNN
-F 2 "" H 7800 4250 60  0001 C CNN
+F 2 "Transistors_TO-220:TO-220_FET-GDS_Vertical" H 7800 4250 60  0001 C CNN
 F 3 "" H 7800 4250 60  0000 C CNN
 F 4 "BUK9575-100A,127" H 7800 4250 60  0001 C CNN "MPN"
@@
 $EndComp
 $Comp
-L GND #PWR209
+L GND #PWR010
 U 1 1 5521A14F
 P 5100 4750
-F 0 "#PWR209" H 5100 4500 60  0001 C CNN
+F 0 "#PWR010" H 5100 4500 60  0001 C CNN
 F 1 "GND" H 5100 4600 60  0000 C CNN
 F 2 "" H 5100 4750 60  0000 C CNN
@@
 $EndComp
 $Comp
-L GND #PWR205
+L GND #PWR011
 U 1 1 5521A15C
 P 4300 3850
-F 0 "#PWR205" H 4300 3600 60  0001 C CNN
+F 0 "#PWR011" H 4300 3600 60  0001 C CNN
 F 1 "GND" H 4300 3700 60  0000 C CNN
 F 2 "" H 4300 3850 60  0000 C CNN
@@
 Connection ~ 3800 4150
 $Comp
-L GND #PWR201
+L GND #PWR012
 U 1 1 5526E331
 P 3800 4900
-F 0 "#PWR201" H 3800 4650 50  0001 C CNN
+F 0 "#PWR012" H 3800 4650 50  0001 C CNN
 F 1 "GND" H 3800 4750 50  0000 C CNN
 F 2 "" H 3800 4900 60  0000 C CNN
@@
 F 0 "P201" H 4250 4650 50  0000 C BNN
 F 1 "TST" H 4250 4600 50  0000 C CNN
-F 2 "" H 4250 4350 60  0000 C CNN
+F 2 "Measurement_Points:Measurement_Point_Round-TH_Small" H 4250 4350 60  0001 C CNN
 F 3 "" H 4250 4350 60  0000 C CNN
 	1    4250 4350
@@
 F 0 "P202" H 8250 5050 50  0000 C BNN
 F 1 "TST" H 8250 5000 50  0000 C CNN
-F 2 "" H 8250 4750 60  0000 C CNN
+F 2 "Measurement_Points:Measurement_Point_Round-TH_Small" H 8250 4750 60  0001 C CNN
 F 3 "" H 8250 4750 60  0000 C CNN
 	1    8250 4750

Commit message: updated schematic with part numbers to ICs
Parts:
- U201: footprint SMD_Packages:SOIC-8-N -> SOIC-8-N; MPN (none) -> LMV358IDT
Changed lines of the file:
@@
 F 0 "U201" H 5150 4450 60  0000 L CNN
 F 1 "LMV358" H 5150 4000 60  0000 L CNN
-F 2 "SMD_Packages:SOIC-8-N" H 5200 4250 60  0001 C CNN
-F 3 "" H 5200 4250 60  0000 C CNN
+F 2 "SOIC-8-N" H 5200 4250 60  0001 C CNN
+F 3 "http://www.st.com/web/en/resource/technical/document/datasheet/CD00079372.pdf" H 5200 4250 60  0001 C CNN
+F 4 "LMV358IDT" H 5200 4250 60  0001 C CNN "MPN"
 	1    5200 4250
 	1    0    0    -1
@@
 F 1 "BUK9575" H 7750 4100 50  0000 R CNN
 F 2 "Transistors_TO-220:TO-220_FET-GDS_Vertical" H 7800 4250 60  0001 C CNN
-F 3 "" H 7800 4250 60  0000 C CNN
+F 3 "http://www.nxp.com/documents/data_sheet/BUK9575_9675-100A.pdf" H 7800 4250 60  0001 C CNN
 F 4 "BUK9575-100A,127" H 7800 4250 60  0001 C CNN "MPN"
 	1    7800 4250
