File: powerRegulation.sch (KiCad schematic (older format))
At the start: 13 parts, among them P401 TST, U401 LM2931, U402 MCP1640T

Commit message: removed duplicates and bad wire connections to enable the generation of a PCB
Parts:
- U401: footprint Power_Integrations:SO-8 -> SO-8
- U402: footprint Housings_SOT-23_SOT-143_TSOT-6:SOT-23-6 -> SOT-23-6
Changed lines of the file:
@@
 F 0 "U402" H 6800 4650 40  0000 C CNN
 F 1 "MCP1640T" H 6800 5200 40  0000 C CNN
-F 2 "Housings_SOT-23_SOT-143_TSOT-6:SOT-23-6" H 6550 4950 30  0000 C CIN
+F 2 "SOT-23-6" H 6550 4950 30  0000 C CIN
 F 3 "" H 6550 4900 60  0000 C CNN
 	1    6550 4900
@@
 F 0 "U401" H 5600 3000 40  0000 C CNN
 F 1 "LM2931" H 5800 3000 40  0000 L CNN
-F 2 "Power_Integrations:SO-8" H 5800 2900 30  0000 C CIN
+F 2 "SO-8" H 5800 2900 30  0000 C CIN
 F 3 "" H 5800 2700 60  0000 C CNN
 	1    5800 2800

Commit message: initial layout complete with gnd plane
Parts:
- U401: footprint SO-8 -> Power_Integrations:SO-8
- U402: footprint SOT-23-6 -> Housings_SOT-23_SOT-143_TSOT-6:SOT-23-6
Changed lines of the file:
@@
 F 0 "U402" H 6800 4650 40  0000 C CNN
 F 1 "MCP1640T" H 6800 5200 40  0000 C CNN
-F 2 "SOT-23-6" H 6550 4950 30  0000 C CIN
+F 2 "Housings_SOT-23_SOT-143_TSOT-6:SOT-23-6" H 6550 4950 30  0000 C CIN
 F 3 "" H 6550 4900 60  0000 C CNN
 	1    6550 4900
@@
 F 0 "U401" H 5600 3000 40  0000 C CNN
 F 1 "LM2931" H 5800 3000 40  0000 L CNN
-F 2 "SO-8" H 5800 2900 30  0000 C CIN
+F 2 "Power_Integrations:SO-8" H 5800 2900 30  0000 C CIN
 F 3 "" H 5800 2700 60  0000 C CNN
 	1    5800 2800

Commit message: updated schematic with part numbers to ICs
Parts:
- U401: footprint Power_Integrations:SO-8 -> SO-8; MPN (none) -> LM2931D-R
- U402: footprint Housings_SOT-23_SOT-143_TSOT-6:SOT-23-6 -> SOT-23-6; MPN (none) -> MCP1640T-I/CHY
Changed lines of the file:
@@
 F 0 "U402" H 6800 4650 40  0000 C CNN
 F 1 "MCP1640T" H 6800 5200 40  0000 C CNN
-F 2 "Housings_SOT-23_SOT-143_TSOT-6:SOT-23-6" H 6550 4950 30  0000 C CIN
-F 3 "" H 6550 4900 60  0000 C CNN
+F 2 "SOT-23-6" H 6550 4950 30  0000 C CIN
+F 3 "http://ww1.microchip.com/downloads/en/DeviceDoc/20002234C.pdf" H 6550 4900 60  0001 C CNN
+F 4 "MCP1640T-I/CHY" H 6550 4900 60  0001 C CNN "MPN"
 	1    6550 4900
 	1    0    0    -1
@@
 F 0 "U401" H 5600 3000 40  0000 C CNN
 F 1 "LM2931" H 5800 3000 40  0000 L CNN
-F 2 "Power_Integrations:SO-8" H 5800 2900 30  0000 C CIN
-F 3 "" H 5800 2700 60  0000 C CNN
+F 2 "SO-8" H 5800 2900 30  0000 C CIN
+F 3 "http://www.st.com/web/en/resource/technical/document/datasheet/CD00001885.pdf" H 5800 2700 60  0001 C CNN
+F 4 "LM2931D-R" H 5800 2800 60  0001 C CNN "MPN"
 	1    5800 2800
 	1    0    0    -1
